Commit message: test_ik

File: install/six_arm/share/six_arm/urdf/cobot.urdf.xacro (robot description, xacro)
@@ -1 +1,162 @@
-/home/fra/master_ws_test/src/six_arm/urdf/cobot.urdf.xacro
+<?xml version = "1.0"?>
+<robot name="custom_robot" xmlns:xacro="http://www.ros.org/wiki/xacro">
+    <xacro:include filename="/home/fra/master_ws_test/src/six_arm/urdf/link_joint.xacro" />
+    <xacro:include filename="/home/fra/master_ws_test/src/six_arm/urdf/custom_gripper.xacro"/>
+    <xacro:include filename="/home/fra/master_ws_test/src/six_arm/urdf/custom_robot_gazebo.xacro"/>
+    <link name="world">
+    </link>
+    <xacro:cobot_link_cylinder name="base_link" origin_xyz="0.0 0.0 0.02" origin_rpy= "0 0 0"
+                            radius="0.05" length="0.04" mass="4" i_xx="0.003033" i_xy="0" i_xz="0"
+                            i_yy="0.003033" i_yz="0" i_zz="0.005" />
+    <joint name="fixed" type="fixed">
+        <parent link="world"/>
+        <child link="base_link"/>
+        <origin xyz="0 0.0 0.8" rpy="0 0 0"/>
+    </joint>
+    <xacro:cobot_link_cylinder name="link1" origin_xyz="0.0 0.0 0.045" origin_rpy= "0 0 0"
+                            radius="0.035" length="0.09" mass="3.7" i_xx="0.003630625" i_xy="0" i_xz="0"
+                            i_yy="0.003630625" i_yz="0" i_zz="0.00226625" />
+    <xacro:cobot_joint name="base_link__link1" type="revolute" parent="base_link" child="link1" axis="0 0 1"
+                        limit_l="-3.14159" limit_u="3.14159" limit_v="0.5" limit_e="1000"
+                        origin_xyz="0 0 0.04" origin_rpy="0 0 0" />
+    <xacro:cobot_link_cylinder name="link2" origin_xyz="0.0 0.0 0.2125" origin_rpy= "0 0 0"
+                            radius="0.035" length="0.425"  mass="8.3" i_xx="0.499729" i_xy="0" i_xz="0"
+                            i_yy="0" i_yz="0" i_zz="0.499729"/>
+    <joint name="link1__link2" type="revolute">
+        <parent link="link1"/>
+        <child link="link2"/>
+        <axis xyz="0 1 0"/>
+        <limit lower="-3.14159" upper="3.14159" velocity="0.5" effort="1000.0"/>
+        <origin xyz="0 0.07 0.055" rpy="0 0 0"/>
+    </joint>
+    <xacro:cobot_link_cylinder name="link3" origin_xyz="0.0 0.0 0.196" origin_rpy= "0 0 0"
+                            radius="0.035" length="0.392" mass="2.3" i_xx="0.117809067" i_xy="0" i_xz="0"
+                            i_yy="0" i_yz="0" i_zz="0.117809067" />
+    <xacro:cobot_joint name="link2__link3" type="revolute" parent="link2" child="link3" axis="0 1 0"
+                        limit_l="-3.14159" limit_u="3.14159" limit_v="0.5" limit_e="1000"
+                        origin_xyz="0 -0.0675 0.39" origin_rpy="0 0 0" />
+    <xacro:cobot_link_cylinder name="link4" origin_xyz="0.0 0.0 0.047" origin_rpy= "0 0 0"
+                            radius="0.035" length="0.094" mass="1.2" i_xx="0.0035344" i_xy="0" i_xz="0"
+                            i_yy="0" i_yz="0" i_zz="0.0035344" />
+    <xacro:cobot_joint name="link3__link4" type="revolute" parent="link3" child="link4" axis="0 1 0"
+                        limit_l="-3.14159" limit_u="3.14159" limit_v="0.5" limit_e="1000"
+                        origin_xyz="0 0.0675 0.357" origin_rpy="0 0 0" />
+    <xacro:cobot_link_cylinder name="link5" origin_xyz="0.0 0.0 0.009" origin_rpy= "0 0 0"
+                            radius="0.0325" length="0.083" mass="1.2" i_xx="0.0027556" i_xy="0" i_xz="0"
+                            i_yy="0" i_yz="0" i_zz="0.0027556" />
+    <xacro:cobot_joint name="link4__link5" type="revolute" parent="link4" child="link5" axis="0 1 0"
+                        limit_l="-3.14159" limit_u="3.14159" limit_v="0.5" limit_e="1000"
+                        origin_xyz="0 0.0 0.1265" origin_rpy="1.57 0 0" />
+    <xacro:cobot_link_cylinder name="link6" origin_xyz="0.0 0.0 0.01" origin_rpy= "0 0 0"
+                            radius="0.0325" length="0.02" mass="0.2" i_xx="0.000059479" i_xy="0" i_xz="0"
+                            i_yy="0.000059479" i_yz="0" i_zz="0.000105625" />
+    <xacro:cobot_joint name="link5__link6" type="revolute" parent="link5" child="link6" axis="0 0 1"
+                        limit_l="-3.14159" limit_u="3.14159" limit_v="0.5" limit_e="1000"
+                        origin_xyz="0 0.0 0.0505" origin_rpy="0 0 0" />
+    <!--put end effector tool-->
+    <link name="tool0">
+    </link>
+    <joint name="link6__tool0" type="fixed">
+        <parent link="link6"/>
+        <child link="tool0"/>
+        <origin xyz="0.0 0.0 0.02" rpy="0.0 0.0 0.0"/>
+    </joint>
+    <link name="picking_point">
+    </link>
+    <joint name="tool0_picking_point" type="fixed">
+        <parent link="tool0"/>
+        <child link="picking_point"/>
+        <origin xyz="0.0 0.0 0.08" rpy="0.0 0.0 0.0"/>
+    </joint>
+    <xacro:custom_gripper parent="tool0" origin_xyz="0 0 0" />
+    <ros2_control name="GazeboSystem" type="system">
+        <hardware>
+            <plugin>gazebo_ros2_control/GazeboSystem</plugin>
+        </hardware>
+        <joint name="base_link__link1">
+            <command_interface name="position">
+                <param name="min">-6.28</param>
+                <param name="max">6.28</param>
+            </command_interface>
+            <state_interface name="position">
+                <param name="initial_value">0.0</param>
+            </state_interface>
+            <state_interface name="velocity" />
+        </joint>
+        <joint name="link1__link2">
+            <command_interface name="position">
+                <param name="min">-6.28</param>
+                <param name="max">6.28</param>
+            </command_interface>
+            <state_interface name="position" >
+                <param name="initial_value">0.0</param>
+            </state_interface>
+            <state_interface name="velocity" />
+        </joint>
+        <joint name="link2__link3">
+            <command_interface name="position">
+                <param name="min">-6.28</param>
+                <param name="max">6.28</param>
+            </command_interface>
+            <state_interface name="position" >
+                <param name="initial_value">0.0</param>
+            </state_interface>
+            <state_interface name="velocity" />
+        </joint>
+        <joint name="link3__link4">
+            <command_interface name="position">
+                <param name="min">-6.28</param>
+                <param name="max">6.28</param>
+            </command_interface>
+            <state_interface name="position" >
+                <param name="initial_value">0.0</param>
+            </state_interface>
+            <state_interface name="velocity" />
+        </joint>
+        <joint name="link4__link5">
+            <command_interface name="position">
+                <param name="min">-6.28</param>
+                <param name="max">6.28</param>
+            </command_interface>
+            <state_interface name="position" >
+                <param name="initial_value">0.0</param>
+            </state_interface>
+            <state_interface name="velocity" />
+        </joint>
+        <joint name="link5__link6">
+            <command_interface name="position">
+                <param name="min">-6.28</param>
+                <param name="max">6.28</param>
+            </command_interface>
+            <state_interface name="position" >
+                <param name="initial_value">0.0</param>
+            </state_interface>
+            <state_interface name="velocity" />
+        </joint>
+        <joint name="finger_right_joint">
+            <command_interface name="position" />
+            <state_interface name="position" >
+                <param name="initial_value">0.0</param>
+            </state_interface>
+            <state_interface name="velocity" />
+        </joint>
+        <joint name="finger_left_joint">
+            <param name="mimic">finger_right_joint</param>
+            <param name="multiplier">-1</param>
+            <command_interface name="position" />
+            <state_interface name="position" >
+                <param name="initial_value">0.0</param>
+            </state_interface>
+            <state_interface name="velocity" />
+        </joint>
+    </ros2_control>
+    <gazebo>
+        <plugin filename="libgazebo_ros2_control.so" name="gazebo_ros2_control">
+            <!-- <ros>
+                <namespace>/cobot</namespace>
+            </ros> -->
+            <robot_param>robot_description</robot_param>
+            <parameters>$(find six_arm)/config/controllers.yaml </parameters>
+        </plugin>
+    </gazebo>
+</robot>

File: install/six_arm/share/six_arm/urdf/custom_gripper.xacro (robot description, xacro)
@@ -1 +1,56 @@
-/home/fra/master_ws_test/src/six_arm/urdf/custom_gripper.xacro
+<?xml version = "1.0"?>
+<robot xmlns:xacro="http://www.ros.org/wiki/xacro">
+    <xacro:include filename="/home/fra/master_ws_test/src/six_arm/urdf/link_joint.xacro"/>
+    <xacro:include filename="/home/fra/master_ws_test/src/six_arm/urdf/custom_robot_gazebo.xacro"/>
+    <!-- Model a gripper-->
+    <xacro:macro name="custom_gripper" params = "parent origin_xyz" >
+        <xacro:cobot_link_cylinder name="gripper_connector" origin_xyz="0.0 0.0 0.015" origin_rpy= "0 0 0"
+                            radius="0.04" length="0.03" mass="0.5" i_xx="0.0002375" i_xy="0" i_xz="0"
+                            i_yy="0.0002375" i_yz="0" i_zz="0.00006666666667" />
+        <joint name="{parent}__gripper_connector" type="fixed">
+            <parent link="${parent}"/>
+            <child link="gripper_connector"/>
+            <origin xyz="${origin_xyz}" rpy="0.0 0.0 0.0"/>
+        </joint>
+        <xacro:cobot_link_box name="finger_support" origin_xyz="0 0.005 0.005" origin_rpy="0 0 0"
+                                size="0.120 0.01 0.01" mass="0.25" i_xx="0.0003" i_xy="0" i_xz="0"
+                            i_yy="0.0003" i_yz="0" i_zz="0.0003"/>
+        <joint name="finger_support__gripper_connector" type="fixed">
+            <parent link="gripper_connector"/>
+            <child link="finger_support"/>
+            <origin xyz="0 0 0.03" rpy="0.0 0.0 0.0"/>
+        </joint>
+        <xacro:cobot_link_box name="finger_right" origin_xyz="0 0 0.04" origin_rpy="0 0 0"
+                                size="0.01 0.01 0.08" mass="0.2" i_xx="0.00042667" i_xy="0" i_xz="0"
+                            i_yy="0.00042667" i_yz="0" i_zz="0.0000083"/>
+        <xacro:cobot_link_box name="finger_left" origin_xyz="0 0 0.04" origin_rpy="0 0 0"
+                                size="0.01 0.01 0.08" mass="0.2" i_xx="0.00042667" i_xy="0" i_xz="0"
+                            i_yy="0.00042667" i_yz="0" i_zz="0.0000083"/>
+        <joint name="finger_right_joint" type="prismatic">
+            <parent link="finger_support"/>
+            <child link="finger_right"/>
+            <axis xyz="1 0 0"/>
+            <limit lower="0" upper="0.044" velocity="0.5" effort="400"/>
+            <origin xyz="-0.05 0.0 0.011" rpy="0 0 0"/>
+            <dynamics damping="1" friction="2"/>
+        </joint>
+        <!-- <xacro:transmission_effort name="trans_finger_right_joint"
+                        joint_name="finger_right_joint"
+                        actuator_name="motor_finger_right_joint" /> -->
+        <joint name="finger_left_joint" type="prismatic">
+            <parent link="finger_support"/>
+            <child link="finger_left"/>
+            <axis xyz="1 0 0"/>
+            <limit lower="-0.044" upper="0" velocity="0.5" effort="400"/>
+            <origin xyz="0.05 0.0 0.011" rpy="0 0 0"/>
+            <!-- <dynamics damping="1" friction="2"/> -->
+            <dynamics friction="2"/>
+            <mimic joint="finger_right_joint" multiplier="-1.0" offset="0" />
+        </joint>
+        <!-- <xacro:transmission_effort name="trans_finger_left_joint"
+                        joint_name="finger_left_joint"
+                        actuator_name="motor_finger_left_joint" /> -->
+        <xacro:mimic_joint_plugin_gazebo  parent_joint="finger_right_joint" mimic_joint="finger_left_joint"
+                                            has_pid="false" multiplier="-1.0" max_effort="200" />
+    </xacro:macro>
+</robot>

File: install/six_arm/share/six_arm/urdf/custom_robot_gazebo.xacro (robot description, xacro)
@@ -1 +1,76 @@
-/home/fra/master_ws_test/src/six_arm/urdf/custom_robot_gazebo.xacro
+<?xml version = "1.0"?>
+<robot xmlns:xacro="http://www.ros.org/wiki/xacro">
+    <!-- Make the robot more fancy :)-->
+    <gazebo reference="base_link" >
+        <material>Gazebo/Blue</material>
+    </gazebo>
+    <gazebo reference="link1" >
+        <material>Gazebo/Yellow</material>
+    </gazebo>
+    <gazebo reference="link2" >
+        <material>Gazebo/Black</material>
+    </gazebo>
+    <gazebo reference="link3" >
+        <material>Gazebo/Yellow</material>
+    </gazebo>
+    <gazebo reference="link4" >
+        <material>Gazebo/Black</material>
+    </gazebo>
+    <gazebo reference="link5" >
+        <material>Gazebo/Yellow</material>
+    </gazebo>
+    <gazebo reference="link6" >
+        <material>Gazebo/Black</material>
+    </gazebo>
+    <gazebo reference="gripper_connector" >
+        <material>Gazebo/Black</material>
+    </gazebo>
+    <gazebo reference="finger_support" >
+        <material>Gazebo/Black</material>
+    </gazebo>
+    <gazebo reference="finger_right" >
+        <material>Gazebo/Blue</material>
+    </gazebo>
+    <gazebo reference="finger_left" >
+        <material>Gazebo/Blue</material>
+    </gazebo>
+    <!-- ros control plugin with mimic-->
+        <xacro:macro name="mimic_joint_plugin_gazebo" params="parent_joint mimic_joint has_pid:=false multiplier:=-1.0 offset:=0 sensitiveness:=0.0 max_effort:=200 robot_namespace:='/cobot'">
+            <gazebo>
+                <plugin name="${mimic_joint}_mimic_joint_plugin" filename="libroboticsgroup_upatras_gazebo_mimic_joint_plugin.so">
+                    <joint>${parent_joint}</joint>
+                    <mimicJoint>${mimic_joint}</mimicJoint>
+                    <xacro:if value="${has_pid}">
+                        <hasPID />
+                    </xacro:if>
+                    <multiplier>${multiplier}</multiplier>
+                    <offset>${offset}</offset>
+                    <sensitiveness>${sensitiveness}</sensitiveness>
+                    <maxEffort>${max_effort}</maxEffort>
+                    <xacro:unless value="${robot_namespace == '/cobot'}">
+                        <robotNamespace>($robot_namespace)</robotNamespace>
+                    </xacro:unless>
+                </plugin>
+            </gazebo>
+        </xacro:macro>
+    <!-- <gazebo>
+        <plugin name="gazebo_grasp_fix" filename="libgazebo_grasp_fix.so">
+            <arm>
+                <arm_name>custom_gripper</arm_name>
+                <palm_link> link6 </palm_link>
+                <gripper_link> finger_right </gripper_link>
+                <gripper_link> finger_left </gripper_link>
+            </arm>
+        <forces_angle_tolerance>100</forces_angle_tolerance>
+        <update_rate>4</update_rate>
+        <grip_count_threshold>4</grip_count_threshold>
+        <max_grip_count>8</max_grip_count>
+        <release_tolerance>0.005</release_tolerance>
+        <disable_collisions_on_attach>false</disable_collisions_on_attach>
+        <contact_topic>__default_topic__</contact_topic>
+        </plugin>
+    </gazebo> -->
+    <gazebo>
+        <plugin name="link_attacher" filename="libgazebo_ros_link_attacher.so"/>
+    </gazebo>
+</robot>

File: install/six_arm/share/six_arm/urdf/link_joint.xacro (robot description, xacro)
@@ -1 +1,54 @@
-/home/fra/master_ws_test/src/six_arm/urdf/link_joint.xacro
+<?xml version = "1.0"?>
+<robot xmlns:xacro="http://www.ros.org/wiki/xacro">
+    <xacro:macro name="cobot_link_cylinder" params="name origin_xyz origin_rpy radius length mass i_xx i_xy i_xz i_yy i_yz i_zz">
+        <link name="${name}">
+            <inertial>
+                <origin xyz="${origin_xyz}" rpy="${origin_rpy}"/>
+                <mass value="${mass}"/>
+                <inertia ixx="${i_xx}" ixy="${i_xy}" ixz="${i_xz}" iyy="${i_yy}" iyz="${i_yz}" izz="${i_zz}"/>
+            </inertial>
+            <visual>
+                <geometry>
+                    <cylinder radius="${radius}" length="${length}"/>
+                </geometry>
+                <origin xyz="${origin_xyz}" rpy="${origin_rpy}"/>
+            </visual>
+            <collision>
+                <geometry>
+                    <cylinder radius="${radius}" length="${length}"/>
+                </geometry>
+                <origin xyz="${origin_xyz}" rpy="${origin_rpy}"/>
+            </collision>
+        </link>
+    </xacro:macro>
+    <xacro:macro name="cobot_link_box" params="name origin_xyz origin_rpy size mass i_xx i_xy i_xz i_yy i_yz i_zz">
+        <link name="${name}">
+            <inertial>
+                <origin xyz="${origin_xyz}" rpy="${origin_rpy}"/>
+                <mass value="${mass}"/>
+                <inertia ixx="${i_xx}" ixy="${i_xy}" ixz="${i_xz}" iyy="${i_yy}" iyz="${i_yz}" izz="${i_zz}"/>
+            </inertial>
+            <visual>
+                <geometry>
+                    <box size="${size}"/>
+                </geometry>
+                <origin xyz="${origin_xyz}" rpy="${origin_rpy}"/>
+            </visual>
+            <collision>
+                <geometry>
+                    <box size="${size}"/>
+                </geometry>
+                <origin xyz="${origin_xyz}" rpy="${origin_rpy}"/>
+            </collision>
+        </link>
+    </xacro:macro>
+    <xacro:macro name="cobot_joint" params="name type parent child axis limit_l limit_u limit_v limit_e origin_xyz origin_rpy">
+        <joint name="${name}" type="${type}">
+            <parent link="${parent}"/>
+            <child link="${child}"/>
+            <axis xyz="${axis}"/>
+            <limit lower="${limit_l}" upper="${limit_u}" velocity="${limit_v}" effort="${limit_e}"/>
+            <origin xyz="${origin_xyz}" rpy="${origin_rpy}"/>
+        </joint>
+    </xacro:macro>
+</robot>

File: src/six_arm/urdf/cobot.urdf.xacro (robot description, xacro)
@@ -151,14 +151,10 @@
         </joint>
     </ros2_control>
-    <!-- <gazebo>
-        <plugin name="gazebo_ros2_control" filename = "libgazebo_ros2_control.so">
-            <parameters>$(find custom_robot_gazebo)/config/joint_controllers.yaml </parameters>
-            <ros debug="true" />
-        </plugin>
-    </gazebo> -->
     <gazebo>
         <plugin filename="libgazebo_ros2_control.so" name="gazebo_ros2_control">
+            <!-- <ros>
+                <namespace>/cobot</namespace>
+            </ros> -->
             <robot_param>robot_description</robot_param>
-            <!-- <robot_param_node>robot_state_publisher</robot_param_node> -->
             <parameters>$(find six_arm)/config/controllers.yaml </parameters>
         </plugin>

File: src/six_arm/urdf/custom_robot_gazebo.xacro (robot description, xacro)
@@ -54,5 +54,5 @@
             </gazebo>
         </xacro:macro>
-    <gazebo>
+    <!-- <gazebo>
         <plugin name="gazebo_grasp_fix" filename="libgazebo_grasp_fix.so">
             <arm>
@@ -70,4 +70,7 @@
         <contact_topic>__default_topic__</contact_topic>
         </plugin>
+    </gazebo> -->
+    <gazebo>
+        <plugin name="link_attacher" filename="libgazebo_ros_link_attacher.so"/>
     </gazebo>
 </robot>
